File: ADBT.sch (KiCad schematic (older format))
At the start: 89 parts, among them J1 ADB1, J2 ADB2, J3 microUSB

Commit message: Schematic sketch done
Parts:
- removed F?: 250mA, stdpads:BelFuse_1206, symbol Device:Polyfuse_Small
- removed J2: ADB2, stdpads:MD-40, symbol GW_Connector:MiniDIN-4
- removed Q?: 2N3904, stdpads:SOT-23, symbol Device:Q_NPN_BCE
- removed R?: 33, stdpads:R_0603, symbol Device:R_Small
- removed RN?: 10k, symbol Device:R_Pack04
- removed SW? (x2): SW_Push, symbol Switch:SW_Push
- removed U?: AP3417C, stdpads:SOT-23-5, symbol GW_Power:AP3417C
- removed Y?: 12M, stdpads:Crystal_HC49-SMD, symbol Device:Crystal_Small
- added C10: 33p, stdpads:C_0603, symbol Device:C_Small
- added C7: 100n, stdpads:C_0603, symbol Device:C_Small
- added F1: 500mA, stdpads:BelFuse_1206, symbol Device:Polyfuse_Small
- added H5, H6, H7, H8: (no value), stdpads:PasteHole_1.152mm_NPTH, symbol Mechanical:MountingHole
- added Q2: MMBT3904, stdpads:SOT-23, symbol Transistor_BJT:MMBT3904
- added R13, R16, R19, R33: 27, stdpads:R_0603, symbol Device:R_Small
- added R14: DNP, stdpads:R_0603, symbol Device:R_Small
- added R17, R18: 1k, stdpads:R_0603, symbol Device:R_Small
- added U3: MP2451DT, stdpads:SOT-23-6, symbol GW_Power:MP2451
- added U5: 74LVC1G74DC, stdpads:NXP_VSSOP-8_2.3x2mm, symbol GW_Logic:741G74DC
- added U6: 74LVC1G14GW, stdpads:SOT-353, symbol 74xGxx:74LVC1G14
- added Y1: 12M, stdpads:Crystal_SMD_3225-4Pin_3.2x2.5mm, symbol Device:Crystal_GND24_Small
- C1, C2: renamed from C?; value 680u -> 470u; footprint (none) -> stdpads:CP_Elec_10mm
- C4: renamed from C?; value 10u -> 2u2; footprint stdpads:C_0805 -> stdpads:C_0603
- D1, D2: renamed from D?; LCSC Part (none) -> C22452
- D3: renamed from D?; footprint (none) -> LED_SMD:LED_0805_2012Metric; LCSC Part (none) -> C84256
- D4: renamed from D?; footprint (none) -> LED_SMD:LED_0805_2012Metric; LCSC Part (none) -> C2297
- D5: renamed from D?; value Blue -> Yellow; footprint (none) -> LED_SMD:LED_0805_2012Metric; LCSC Part (none) -> C2296
- D6: renamed from D?; value 6V -> 5V6; footprint (none) -> stdpads:D_MiniMELF; LCSC Part (none) -> C8062
- F2: renamed from F1; LCSC Part (none) -> C69688
- FB1, FB2: renamed from FB?; value BLM21PG300SN1D -> GZ2012D101TF; LCSC Part (none) -> C1015
- H1, H2, H3, H4: footprint stdpads:PasteHole_1.152mm_NPTH -> stdpads:LPSeries-Screw
- J2: renamed from J3; footprint (none) -> stdpads:USB_Micro-B_ShouHan_MicroXNJ; LCSC Part (none) -> C404969
- L1: renamed from L?; footprint (none) -> stdpads:Sunlord_MWSA0402; LCSC Part (none) -> C408335
- Q1: renamed from Q?; LCSC Part (none) -> C15127
- Q3, Q4, Q5: renamed from Q?; value 2N3904 -> MMBT3904; symbol Device:Q_NPN_BCE -> Transistor_BJT:MMBT3904; LCSC Part (none) -> C20526
- R1: renamed from R?; value R -> 124k
- R10, R11, R12: renamed from R?; value 220 -> 100
- R15: renamed from R?; value 1M -> 22k; footprint (none) -> stdpads:R_0603
- R2, R30: renamed from R?; value 33 -> 27
- R3: renamed from R?; value R -> 40.2k
- SW1, SW2: renamed from SW?; footprint (none) -> stdpads:XKB_TS-1187A; LCSC Part (none) -> C480267
- U1: renamed from U?; footprint stdpads:ESP-WROOM-32 -> stdpads:ESP32-WROVER_WROOM-32; LCSC Part (none) -> C473012
- U2: renamed from U?; LCSC Part (none) -> C14267
- U4: renamed from U?; value 74LVC1G14 -> 74LVC1G14GW; LCSC Part (none) -> C265125
- gave numbers to parts that had none: 40
Connections:
- net labels added: ADBsync, BCK, ~BCK~
- net labels removed: BTN2, BTN3
- wire segments 209 -> 210
- no-connect marks 14 -> 15
Other:
- note added: "ADB input receiver & synchronizer"
- note removed: "ADB input receiver"
- moved on the sheet: C1, C13, C14, C15, C16, C17, C18, C19, C2, C20, C21, C22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
